File: pcb/datapack-tool1/datapack-tool1.sch (KiCad schematic (older format))
At the start: 4 parts

Commit message: Updates
Connections:
- net labels added: +3V3, SD0, SD1, SD2, SD3, SD4, SD5, SD6, SD7
- wire segments 3 -> 26
Changed lines of the file:
@@
 U 1 1 63677927
 P 4850 2325
-F 0 "U?" H 4850 3306 50  0000 C CNN
-F 1 "74LS245" H 4850 3215 50  0000 C CNN
+F 0 "U?" H 5100 3325 50  0000 C CNN
+F 1 "74LS245" H 5225 3250 50  0000 C CNN
 F 2 "" H 4850 2325 50  0001 C CNN
 F 3 "http://www.ti.com/lit/gpn/sn74LS245" H 4850 2325 50  0001 C CNN
@@
 U 1 1 63678AE8
 P 4900 4675
-F 0 "U?" H 4900 5656 50  0000 C CNN
-F 1 "74LS245" H 4900 5565 50  0000 C CNN
+F 0 "U?" H 5750 5650 50  0000 C CNN
+F 1 "74LS245" H 5850 5550 50  0000 C CNN
 F 2 "" H 4900 4675 50  0001 C CNN
 F 3 "http://www.ti.com/lit/gpn/sn74LS245" H 4900 4675 50  0001 C CNN
@@
 	1    0    0    -1
 $EndComp
+$Comp
+L power:GND #PWR?
+U 1 1 6367C304
+P 2325 4350
+F 0 "#PWR?" H 2325 4100 50  0001 C CNN
+F 1 "GND" H 2330 4177 50  0000 C CNN
+F 2 "" H 2325 4350 50  0001 C CNN
+F 3 "" H 2325 4350 50  0001 C CNN
+	1    2325 4350
+	1    0    0    -1
+$EndComp
+$Comp
+L power:GND #PWR?
+U 1 1 6367C6EB
+P 4850 3250
+F 0 "#PWR?" H 4850 3000 50  0001 C CNN
+F 1 "GND" H 4855 3077 50  0000 C CNN
+F 2 "" H 4850 3250 50  0001 C CNN
+F 3 "" H 4850 3250 50  0001 C CNN
+	1    4850 3250
+	1    0    0    -1
+$EndComp
+$Comp
+L power:GND #PWR?
+U 1 1 6367CA98
+P 4900 5625
+F 0 "#PWR?" H 4900 5375 50  0001 C CNN
+F 1 "GND" H 4905 5452 50  0000 C CNN
+F 2 "" H 4900 5625 50  0001 C CNN
+F 3 "" H 4900 5625 50  0001 C CNN
+	1    4900 5625
+	1    0    0    -1
+$EndComp
+$Comp
+L power:+3V3 #PWR?
+U 1 1 6367D4B6
+P 3425 1850
+F 0 "#PWR?" H 3425 1700 50  0001 C CNN
+F 1 "+3V3" H 3440 2023 50  0000 C CNN
+F 2 "" H 3425 1850 50  0001 C CNN
+F 3 "" H 3425 1850 50  0001 C CNN
+	1    3425 1850
+	1    0    0    -1
+$EndComp
+$Comp
+L power:+3V3 #PWR?
+U 1 1 6367D50D
+P 4900 3725
+F 0 "#PWR?" H 4900 3575 50  0001 C CNN
+F 1 "+3V3" H 4915 3898 50  0000 C CNN
+F 2 "" H 4900 3725 50  0001 C CNN
+F 3 "" H 4900 3725 50  0001 C CNN
+	1    4900 3725
+	1    0    0    -1
+$EndComp
+$Comp
+L power:+3V3 #PWR?
+U 1 1 6367D984
+P 4850 1275
+F 0 "#PWR?" H 4850 1125 50  0001 C CNN
+F 1 "+3V3" H 4865 1448 50  0000 C CNN
+F 2 "" H 4850 1275 50  0001 C CNN
+F 3 "" H 4850 1275 50  0001 C CNN
+	1    4850 1275
+	1    0    0    -1
+$EndComp
+Wire Wire Line
+	4850 1275 4850 1525
+Wire Wire Line
+	3425 1850 3425 2375
+Wire Wire Line
+	3425 2375 3025 2375
+Wire Wire Line
+	4850 3125 4850 3250
+Wire Wire Line
+	4900 5475 4900 5625
+Wire Wire Line
+	4900 3725 4900 3875
+Wire Wire Line
+	2325 4075 2325 4350
+$Comp
+L power:GND #PWR?
+U 1 1 63680DDA
+P 1325 4350
+F 0 "#PWR?" H 1325 4100 50  0001 C CNN
+F 1 "GND" H 1330 4177 50  0000 C CNN
+F 2 "" H 1325 4350 50  0001 C CNN
+F 3 "" H 1325 4350 50  0001 C CNN
+	1    1325 4350
+	1    0    0    -1
+$EndComp
+$Comp
+L power:GND #PWR?
+U 1 1 6368129A
+P 3475 4350
+F 0 "#PWR?" H 3475 4100 50  0001 C CNN
+F 1 "GND" H 3480 4177 50  0000 C CNN
+F 2 "" H 3475 4350 50  0001 C CNN
+F 3 "" H 3475 4350 50  0001 C CNN
+	1    3475 4350
+	1    0    0    -1
+$EndComp
+Wire Wire Line
+	1325 4350 1325 3675
+Wire Wire Line
+	1325 3675 1625 3675
+Wire Wire Line
+	1625 3175 1325 3175
+Wire Wire Line
+	1325 3175 1325 3675
+Connection ~ 1325 3675
+Wire Wire Line
+	3475 4325 3475 3675
+Wire Wire Line
+	3475 3675 3025 3675
+Wire Wire Line
+	3475 3675 3475 3175
+Wire Wire Line
+	3475 3175 3025 3175
+Connection ~ 3475 3675
+Wire Wire Line
+	3475 3150 3475 2675
+Wire Wire Line
+	3475 2675 3025 2675
+Wire Wire Line
+	1325 3175 1325 2675
+Wire Wire Line
+	1325 2675 1625 2675
+Connection ~ 1325 3175
+Wire Wire Line
+	1625 2175 1325 2175
+Wire Wire Line
+	1325 2175 1325 2675
+Connection ~ 1325 2675
+Wire Wire Line
+	3025 2175 3475 2175
+Wire Wire Line
+	3475 2175 3475 2675
+Connection ~ 3475 2675
+Text GLabel 5350 1825 2    50   Input ~ 0
+P_SD0
+Text GLabel 5350 1925 2    50   Input ~ 0
+P_SD1
+Text GLabel 5350 2025 2    50   Input ~ 0
+P_SD2
+Text GLabel 5350 2125 2    50   Input ~ 0
+P_SD3
+Text GLabel 5350 2225 2    50   Input ~ 0
+P_SD4
+Text GLabel 5350 2325 2    50   Input ~ 0
+P_SD5
+Text GLabel 5350 2425 2    50   Input ~ 0
+P_SD6
+Text GLabel 5350 2525 2    50   Input ~ 0
+P_SD7
+Text GLabel 4350 1825 0    50   Input ~ 0
+SD0
+Text GLabel 4350 1925 0    50   Input ~ 0
+SD1
+Text GLabel 4350 2025 0    50   Input ~ 0
+SD2
+Text GLabel 4350 2125 0    50   Input ~ 0
+SD3
+Text GLabel 4350 2225 0    50   Input ~ 0
+SD4
+Text GLabel 4350 2325 0    50   Input ~ 0
+SD5
+Text GLabel 4350 2425 0    50   Input ~ 0
+SD6
+Text GLabel 4350 2525 0    50   Input ~ 0
+SD7
 $EndSCHEMATC

Commit message: Updates
Connections:
- net labels added: SCLK, SMR, SOE, SPGM, SS
Changed lines of the file:
@@
 Text GLabel 4350 2525 0    50   Input ~ 0
 SD7
+Text GLabel 1625 1975 0    50   Input ~ 0
+SD0
+Text GLabel 1625 2075 0    50   Input ~ 0
+SD1
+Text GLabel 1625 2275 0    50   Input ~ 0
+SD2
+Text GLabel 1625 2375 0    50   Input ~ 0
+SD3
+Text GLabel 1625 2475 0    50   Input ~ 0
+SD4
+Text GLabel 1625 2575 0    50   Input ~ 0
+SD5
+Text GLabel 1625 2775 0    50   Input ~ 0
+SD6
+Text GLabel 1625 2875 0    50   Input ~ 0
+SD7
+Text GLabel 5400 4175 2    50   Input ~ 0
+P_SMR
+Text GLabel 5400 4275 2    50   Input ~ 0
+P_SOE
+Text GLabel 5400 4575 2    50   Input ~ 0
+P_SCLK
+Text GLabel 5400 4475 2    50   Input ~ 0
+P_SS1
+Text GLabel 5400 4375 2    50   Input ~ 0
+P_SPGM
+Text GLabel 4400 4175 0    50   Input ~ 0
+SMR
+Text GLabel 4400 4275 0    50   Input ~ 0
+SOE
+Text GLabel 4400 4375 0    50   Input ~ 0
+SPGM
+Text GLabel 4400 4475 0    50   Input ~ 0
+SS
+Text GLabel 4400 4575 0    50   Input ~ 0
+SCLK
+Text GLabel 1625 2975 0    50   Input ~ 0
+SMR
+Text GLabel 1625 3075 0    50   Input ~ 0
+SOE
+Text GLabel 1625 3275 0    50   Input ~ 0
+SPGM
+Text GLabel 1625 3375 0    50   Input ~ 0
+SS
+Text GLabel 1625 3475 0    50   Input ~ 0
+SCLK
 $EndSCHEMATC

Commit message: Updates
Parts:
- added J?: Conn_01x04_Female, ajm_kicad:OLED_SMALL, symbol Connector:Conn_01x04_Female
- added J?: Conn_01x03_Female, symbol Connector:Conn_01x03_Female
- added M?: P-CHANNEL-MOSFET, Package_TO_SOT_SMD:SOT-23, symbol GeekAmmo:P-CHANNEL-MOSFET
- added R?: 10k, Resistor_SMD:R_0805_2012Metric, symbol Device:R_Small
- added R? (x2): R_Small, Capacitor_SMD:C_0402_1005Metric, symbol Device:R_Small
- added SW? (x4): sw, Button_Switch_SMD:SW_Push_1P1T_NO_Vertical_Wuerth_434133025816, symbol mirotan-due-cassette-shield-cache:Switch_SW_SPST
- added TR?: Si2302CDS-n-channel, Package_TO_SOT_SMD:SOT-23, symbol New_Library:Si2302CDS-n-channel
- added XS?: 502p_SD_ebay-uSD-push_push_SMD, Connectors:Conn_uSDcard, symbol pak_breakout:502p_SD_ebay-uSD-push_push_SMD
Connections:
- net labels added: 5V, 5V_ON, DATA_DIR, I2C_SCLK, I2C_SDA, MISO_D0, MOSI_DI, SD_CLK, SD_DAT1, SD_DAT2, SD_SS, SW0, SW1, SW2, SW3, SWCLK, SWDIO
- wire segments 26 -> 87
Other:
- note added: "Internal pull-ups"
- moved on the sheet: U?

Commit message: Updates
Parts:
- added R?: 10k, symbol Device:R_Small
- R? (x2): value R_Small -> 4k7
Connections:
- net 5V_ON is gone; now on net VPP_ON: TR?.1 (G)
- net GND: now also R?.2
- net SW0: now also U?.34 (GPIO28_ADC2)
- net SW1: now also U?.32 (GPIO27_ADC1)
- net SW2: now also U?.31 (GPIO26_ADC0)
- net VCC_SLOT: no longer M?.3 (D)
- net VPP_DRIVE: now also M?.3 (D)
- net VPP_ON: now reaches U?.22 (GPIO17)
- net VPP_ON: now also R?.1
- net VPP_IN: now reaches U?.40 (VBUS)
- net 5V renamed VPP_SUPPLY
Other:
- moved on the sheet: J?
Changed lines of the file:
@@
 $Descr A4 11693 8268
 encoding utf-8
-Sheet 1 4
+Sheet 1 2
 Title ""
 Date ""
@@
 	1    0    0    -1
 $EndComp
-$Sheet
-S 6100 750  1325 500
-U 6366C142
-F0 "Sheet6366C141" 50
-F1 "org2power.sch" 50
-$EndSheet
 $Comp
 L Connector_Generic:Conn_02x08_Odd_Even J?
 U 1 1 636773E8
-P 8775 2475
+P 10075 2075
 AR Path="/6366C142/636773E8" Ref="J?"  Part="1"
 AR Path="/636773E8" Ref="J?"  Part="1"
-F 0 "J?" H 8825 2992 50  0000 C CNN
-F 1 "Conn_02x08_Odd_Even" H 8825 2901 50  0000 C CNN
-F 2 "ajm_kicad:PinHeader_2x08_P2.54mm_Horizontal_psionSide" H 8775 2475 50  0001 C CNN
-F 3 "~" H 8775 2475 50  0001 C CNN
-	1    8775 2475
-	1    0    0    -1
-$EndComp
-Text GLabel 9075 2175 2    50   Input ~ 0
+F 0 "J?" H 10125 2592 50  0000 C CNN
+F 1 "Conn_02x08_Odd_Even" H 10125 2501 50  0000 C CNN
+F 2 "ajm_kicad:PinHeader_2x08_P2.54mm_Horizontal_psionSide" H 10075 2075 50  0001 C CNN
+F 3 "~" H 10075 2075 50  0001 C CNN
+	1    10075 2075
+	1    0    0    -1
+$EndComp
+Text GLabel 10375 1775 2    50   Input ~ 0
 P_SD0
-Text GLabel 8575 2175 0    50   Input ~ 0
+Text GLabel 9875 1775 0    50   Input ~ 0
 P_SD1
-Text GLabel 9075 2275 2    50   Input ~ 0
+Text GLabel 10375 1875 2    50   Input ~ 0
 P_SD2
-Text GLabel 8575 2275 0    50   Input ~ 0
+Text GLabel 9875 1875 0    50   Input ~ 0
 P_SD3
-Text GLabel 9075 2375 2    50   Input ~ 0
+Text GLabel 10375 1975 2    50   Input ~ 0
 P_SD4
-Text GLabel 8575 2375 0    50   Input ~ 0
+Text GLabel 9875 1975 0    50   Input ~ 0
 P_SD5
-Text GLabel 9075 2475 2    50   Input ~ 0
+Text GLabel 10375 2075 2    50   Input ~ 0
 P_SD6
-Text GLabel 8575 2475 0    50   Input ~ 0
+Text GLabel 9875 2075 0    50   Input ~ 0
 P_SD7
-Text GLabel 8575 2575 0    50   Input ~ 0
+Text GLabel 9875 2175 0    50   Input ~ 0
 P_SMR
-Text GLabel 9075 2575 2    50   Input ~ 0
+Text GLabel 10375 2175 2    50   Input ~ 0
 P_SCLK
-Text GLabel 8575 2675 0    50   Input ~ 0
+Text GLabel 9875 2275 0    50   Input ~ 0
 P_SOE
-Text GLabel 9075 2675 2    50   Input ~ 0
+Text GLabel 10375 2275 2    50   Input ~ 0
 P_SS1
 $Comp
 L power:GND #PWR?
 U 1 1 636773FA
-P 8350 3100
+P 9650 2700
 AR Path="/6366C142/636773FA" Ref="#PWR?"  Part="1"
 AR Path="/636773FA" Ref="#PWR?"  Part="1"
-F 0 "#PWR?" H 8350 2850 50  0001 C CNN
-F 1 "GND" H 8355 2927 50  0000 C CNN
-F 2 "" H 8350 3100 50  0001 C CNN
-F 3 "" H 8350 3100 50  0001 C CNN
-	1    8350 3100
-	1    0    0    -1
-$EndComp
-Wire Wire Line
-	8350 2775 8575 2775
-Wire Wire Line
-	8350 2775 8350 3100
-Text GLabel 8050 2875 0    50   Input ~ 0
+F 0 "#PWR?" H 9650 2450 50  0001 C CNN
+F 1 "GND" H 9655 2527 50  0000 C CNN
+F 2 "" H 9650 2700 50  0001 C CNN
+F 3 "" H 9650 2700 50  0001 C CNN
+	1    9650 2700
+	1    0    0    -1
+$EndComp
+Wire Wire Line
+	9650 2375 9875 2375
+Wire Wire Line
+	9650 2375 9650 2700
+Text GLabel 9350 2475 0    50   Input ~ 0
 VCC_SLOT
 Wire Wire Line
-	8575 2875 8050 2875
-Text GLabel 9075 2775 2    50   Input ~ 0
+	9875 2475 9350 2475
+Text GLabel 10375 2375 2    50   Input ~ 0
 P_SPGM
-Text GLabel 9075 2875 2    50   Input ~ 0
+Text GLabel 10375 2475 2    50   Input ~ 0
 VPP_DRIVE
 $Comp
@@
 U 1 1 63678AE8
 P 4900 4675
-F 0 "U?" H 5750 5650 50  0000 C CNN
-F 1 "74LS245" H 5850 5550 50  0000 C CNN
+F 0 "U?" H 5100 5600 50  0000 C CNN
+F 1 "74LS245" H 5225 5475 50  0000 C CNN
 F 2 "" H 4900 4675 50  0001 C CNN
 F 3 "http://www.ti.com/lit/gpn/sn74LS245" H 4900 4675 50  0001 C CNN
@@
 $EndComp
 Text GLabel 8700 3925 0    50   Input ~ 0
-5V
+VPP_SUPPLY
 $Comp
 L Device:R_Small R?
@@
 L power:GND #PWR?
 U 1 1 63690539
-P 9175 5950
+P 9175 6025
 AR Path="/6366C142/63690539" Ref="#PWR?"  Part="1"
 AR Path="/63690539" Ref="#PWR?"  Part="1"
-F 0 "#PWR?" H 9175 5700 50  0001 C CNN
-F 1 "GND" H 9180 5777 50  0000 C CNN
-F 2 "" H 9175 5950 50  0001 C CNN
-F 3 "" H 9175 5950 50  0001 C CNN
-	1    9175 5950
-	1    0    0    -1
-$EndComp
-Wire Wire Line
-	9175 5950 9175 5700
+F 0 "#PWR?" H 9175 5775 50  0001 C CNN
+F 1 "GND" H 9180 5852 50  0000 C CNN
+F 2 "" H 9175 6025 50  0001 C CNN
+F 3 "" H 9175 6025 50  0001 C CNN
+	1    9175 6025
+	1    0    0    -1
+$EndComp
 Text GLabel 10225 5200 2    50   Input ~ 0
-VCC_SLOT
+VPP_DRIVE
 Wire Wire Line
 	9900 4850 9900 5200
 Wire Wire Line
 	9900 5200 10225 5200
-Text GLabel 8575 5500 0    50   Input ~ 0
-5V_ON
-Wire Wire Line
-	8575 5500 8875 5500
-$Sheet
-S 7825 775  950  375
-U 63690FA3
-F0 "Sheet63690FA2" 50
-F1 "picopak.sch" 50
-$EndSheet
 $Comp
 L Connector:Conn_01x04_Female J?
@@
 Wire Wire Line
 	1175 6875 2050 6875
-Text Notes 2000 6350 0    50   ~ 0
-Internal pull-ups
 $Comp
 L Device:R_Small R?
@@
 AR Path="/636A2843" Ref="R?"  Part="1"
 F 0 "R?" H 2109 6696 50  0000 L CNN
-F 1 "R_Small" H 2109 6605 50  0000 L CNN
+F 1 "4k7" H 2109 6605 50  0000 L CNN
 F 2 "Capacitor_SMD:C_0402_1005Metric" H 2050 6650 50  0001 C CNN
 F 3 "~" H 2050 6650 50  0001 C CNN
@@
 AR Path="/636A2849" Ref="R?"  Part="1"
 F 0 "R?" H 2609 6696 50  0000 L CNN
-F 1 "R_Small" H 2609 6605 50  0000 L CNN
+F 1 "4k7" H 2609 6605 50  0000 L CNN
 F 2 "Capacitor_SMD:C_0402_1005Metric" H 2550 6650 50  0001 C CNN
 F 3 "~" H 2550 6650 50  0001 C CNN
@@
 U 1 1 636A9B98
 P 3925 7225
+AR Path="/63690FA3/636A9B98" Ref="#PWR?"  Part="1"
+AR Path="/636A9B98" Ref="#PWR?"  Part="1"
 F 0 "#PWR?" H 3925 6975 50  0001 C CNN
 F 1 "GND" H 3930 7052 50  0000 C CNN
@@
 U 1 1 636A9B9E
 P 4600 7225
+AR Path="/63690FA3/636A9B9E" Ref="#PWR?"  Part="1"
+AR Path="/636A9B9E" Ref="#PWR?"  Part="1"
 F 0 "#PWR?" H 4600 6975 50  0001 C CNN
 F 1 "GND" H 4605 7052 50  0000 C CNN
@@
 U 1 1 636A9BA4
 P 5275 7225
+AR Path="/63690FA3/636A9BA4" Ref="#PWR?"  Part="1"
+AR Path="/636A9BA4" Ref="#PWR?"  Part="1"
 F 0 "#PWR?" H 5275 6975 50  0001 C CNN
 F 1 "GND" H 5280 7052 50  0000 C CNN
@@
 U 1 1 636A9BAA
 P 5975 7225
+AR Path="/63690FA3/636A9BAA" Ref="#PWR?"  Part="1"
+AR Path="/636A9BAA" Ref="#PWR?"  Part="1"
 F 0 "#PWR?" H 5975 6975 50  0001 C CNN
 F 1 "GND" H 5980 7052 50  0000 C CNN
@@
 	3175 1550 3175 2050
 Connection ~ 3175 2050
+Text GLabel 8100 5500 0    50   Input ~ 0
+VPP_ON
+$Comp
+L Device:R_Small R?
+U 1 1 636F0992
+P 8525 5875
+F 0 "R?" H 8584 5921 50  0000 L CNN
+F 1 "10k" H 8584 5830 50  0000 L CNN
+F 2 "" H 8525 5875 50  0001 C CNN
+F 3 "~" H 8525 5875 50  0001 C CNN
+	1    8525 5875
+	1    0    0    -1
+$EndComp
+$Comp
+L power:GND #PWR?
+U 1 1 636F1ABE
+P 8525 6050
+AR Path="/6366C142/636F1ABE" Ref="#PWR?"  Part="1"
+AR Path="/636F1ABE" Ref="#PWR?"  Part="1"
+F 0 "#PWR?" H 8525 5800 50  0001 C CNN
+F 1 "GND" H 8530 5877 50  0000 C CNN
+F 2 "" H 8525 6050 50  0001 C CNN
+F 3 "" H 8525 6050 50  0001 C CNN
+	1    8525 6050
+	1    0    0    -1
+$EndComp
+Wire Wire Line
+	9175 5700 9175 6025
+Wire Wire Line
+	8525 6050 8525 5975
+Wire Wire Line
+	8100 5500 8525 5500
+Wire Wire Line
+	8525 5775 8525 5500
+Connection ~ 8525 5500
+Wire Wire Line
+	8525 5500 8875 5500
+Text GLabel 2725 2650 2    50   Input ~ 0
+VPP_ON
+$Sheet
+S 6875 1675 1000 575
+U 63706713
+F0 "Sheet63706712" 50
+F1 "usb.sch" 50
+$EndSheet
+Text GLabel 3375 850  2    50   Input ~ 0
+VPP_IN
+Wire Wire Line
+	2725 850  3375 850
+Text GLabel 3375 1450 2    50   Input ~ 0
+SW0
+Wire Wire Line
+	3375 1450 2725 1450
+Text GLabel 3375 1650 2    50   Input ~ 0
+SW1
+Wire Wire Line
+	3375 1650 2725 1650
+Text GLabel 3375 1750 2    50   Input ~ 0
+SW2
+Wire Wire Line
+	3375 1750 2725 1750
 $EndSCHEMATC

Commit message: Updates
Parts:
- removed SW?: sw, Button_Switch_SMD:SW_Push_1P1T_NO_Vertical_Wuerth_434133025816, symbol mirotan-due-cassette-shield-cache:Switch_SW_SPST
Changed lines of the file:
@@
 Text GLabel 5675 6675 2    50   Input ~ 0
 SW2
-Wire Wire Line
-	5975 7075 5975 7225
-$Comp
-L mirotan-due-cassette-shield-cache:Switch_SW_SPST SW?
-U 1 1 636A9B90
-P 5975 6875
-AR Path="/6104FF77/636A9B90" Ref="SW?"  Part="1"
-AR Path="/636A9B90" Ref="SW?"  Part="1"
-AR Path="/63690FA3/636A9B90" Ref="SW?"  Part="1"
-F 0 "SW?" V 5929 6973 50  0000 L CNN
-F 1 "sw" V 6020 6973 50  0000 L CNN
-F 2 "Button_Switch_SMD:SW_Push_1P1T_NO_Vertical_Wuerth_434133025816" H 5975 6875 50  0001 C CNN
-F 3 "" H 5975 6875 50  0001 C CNN
-	1    5975 6875
-	0    1    1    0
-$EndComp
-Text GLabel 6375 6675 2    50   Input ~ 0
-SW3
-Wire Wire Line
-	6375 6675 5975 6675
 $Comp
 L power:GND #PWR?
@@
 	1    0    0    -1
 $EndComp
-$Comp
-L power:GND #PWR?
-U 1 1 636A9BAA
-P 5975 7225
-AR Path="/63690FA3/636A9BAA" Ref="#PWR?"  Part="1"
-AR Path="/636A9BAA" Ref="#PWR?"  Part="1"
-F 0 "#PWR?" H 5975 6975 50  0001 C CNN
-F 1 "GND" H 5980 7052 50  0000 C CNN
-F 2 "" H 5975 7225 50  0001 C CNN
-F 3 "" H 5975 7225 50  0001 C CNN
-	1    5975 7225
-	1    0    0    -1
-$EndComp

Commit message: Updates
Parts:
- added JP1, JP2, JP3, JP4: Jumper_NO_Small, Jumper:SolderJumper-2_P1.3mm_Open_TrianglePad1.0x1.5mm, symbol Device:Jumper_NO_Small
- added R3, R4, R5, R8: R_Small, Resistor_SMD:R_0805_2012Metric, symbol Device:R_Small
- J1: renamed from J?; footprint ajm_kicad:OLED_SMALL -> Connector_PinHeader_2.54mm:PinHeader_1x04_P2.54mm_Vertical
- J3: renamed from J?; footprint (none) -> Connector_PinHeader_2.54mm:PinHeader_1x03_P2.54mm_Vertical
- R6: renamed from R?; footprint (none) -> Resistor_SMD:R_0805_2012Metric
- U1: renamed from U?; footprint RPi_Pico:RPi_Pico_SMD_TH -> rp2040:RPi_Pico_SMD_TH
- U2, U3: renamed from U?; footprint (none) -> Package_SO:SOP-20_7.5x12.8mm_P1.27mm
- XS1: renamed from XS?; footprint Connectors:Conn_uSDcard -> ajm_kicad:Conn_uSDcard
- gave numbers to parts that had none: 9
Connections:
- net +3V3: now also JP1.2, JP3.2, R3.1, R4.1, R5.1; no longer J1.3 (Pin_3), U3.1 (A->B)
- net GND: now also U3.1 (A->B), JP2.2, JP4.2; no longer J1.4 (Pin_4)
- net SW0: now also R3.2
- net SW1: now also R4.2
- net SW2: now also R5.2
- net at M1.1 (G), R7.2: now also R8.1; no longer TR1.3 (D)
- new net: R8.2, TR1.3 (D)
- new net: J1.3 (Pin_3), JP1.1, JP2.1
- new net: J1.4 (Pin_4), JP3.1, JP4.1
Other:
- note removed: "Internal pull-ups"
- moved on the sheet: J1, R1, R2

Commit message: Updates
Parts:
- added C1, C2: 100nF, Capacitor_SMD:C_0805_2012Metric, symbol Device:C_Small
- added JP5, JP6: Jumper_NO_Small, Jumper:SolderJumper-2_P1.3mm_Open_TrianglePad1.0x1.5mm, symbol Device:Jumper_NO_Small
- added U4: AMS1117-3.3, Package_TO_SOT_SMD:SOT-223-3_TabPin2, symbol pak_breakout:AMS1117-3.3
Connections:
- net +3V3: now also JP5.1, JP6.2; no longer U1.36 (3V3)
- net GND: now also C1.2, C2.2, U4.1 (GND)
- net VPP_IN: now also C1.1, U4.3 (VI)
- new net: JP5.2, U1.36 (3V3)
- new net: C2.1, JP6.1, U4.2 (VO)
Changed lines of the file:
@@
 L power:GND #PWR0103
 U 1 1 6367C6EB
-P 4850 3250
-F 0 "#PWR0103" H 4850 3000 50  0001 C CNN
-F 1 "GND" H 4855 3077 50  0000 C CNN
-F 2 "" H 4850 3250 50  0001 C CNN
-F 3 "" H 4850 3250 50  0001 C CNN
-	1    4850 3250
+P 6575 1300
+F 0 "#PWR0103" H 6575 1050 50  0001 C CNN
+F 1 "GND" H 6580 1127 50  0000 C CNN
+F 2 "" H 6575 1300 50  0001 C CNN
+F 3 "" H 6575 1300 50  0001 C CNN
+	1    6575 1300
 	1    0    0    -1
 $EndComp
@@
 L power:+3V3 #PWR0105
 U 1 1 6367D4B6
-P 3125 725
-F 0 "#PWR0105" H 3125 575 50  0001 C CNN
-F 1 "+3V3" H 3140 898 50  0000 C CNN
-F 2 "" H 3125 725 50  0001 C CNN
-F 3 "" H 3125 725 50  0001 C CNN
-	1    3125 725
+P 4250 850
+F 0 "#PWR0105" H 4250 700 50  0001 C CNN
+F 1 "+3V3" H 4265 1023 50  0000 C CNN
+F 2 "" H 4250 850 50  0001 C CNN
+F 3 "" H 4250 850 50  0001 C CNN
+	1    4250 850
 	1    0    0    -1
 $EndComp
@@
 	4850 1275 4850 1525
 Wire Wire Line
-	3125 725  3125 1250
-Wire Wire Line
-	3125 1250 2725 1250
+	4250 1250 2725 1250
 Wire Wire Line
 	4850 3125 4850 3250
@@
 VPP_IN
 Wire Wire Line
-	2725 850  3375 850
+	2725 850  3075 850
 Text GLabel 3375 1450 2    50   Input ~ 0
 SW0
@@
 Wire Wire Line
 	975  6975 3000 6975
+$Comp
+L Device:Jumper_NO_Small JP5
+U 1 1 63745F7B
+P 4250 1150
+F 0 "JP5" V 4204 1198 50  0000 L CNN
+F 1 "Jumper_NO_Small" V 4295 1198 50  0000 L CNN
+F 2 "Jumper:SolderJumper-2_P1.3mm_Open_TrianglePad1.0x1.5mm" H 4250 1150 50  0001 C CNN
+F 3 "~" H 4250 1150 50  0001 C CNN
+	1    4250 1150
+	0    1    1    0
+$EndComp
+$Comp
+L Device:Jumper_NO_Small JP6
+U 1 1 63746CAC
+P 7150 875
+F 0 "JP6" H 7150 1060 50  0000 C CNN
+F 1 "Jumper_NO_Small" H 7150 969 50  0000 C CNN
+F 2 "Jumper:SolderJumper-2_P1.3mm_Open_TrianglePad1.0x1.5mm" H 7150 875 50  0001 C CNN
+F 3 "~" H 7150 875 50  0001 C CNN
+	1    7150 875
+	1    0    0    -1
+$EndComp
+Wire Wire Line
+	4250 850  4250 1050
+$Comp
+L pak_breakout:AMS1117-3.3 U4
+U 1 1 6374C131
+P 6575 875
+F 0 "U4" H 6575 1117 50  0000 C CNN
+F 1 "AMS1117-3.3" H 6575 1026 50  0000 C CNN
+F 2 "Package_TO_SOT_SMD:SOT-223-3_TabPin2" H 6575 1075 50  0001 C CNN
+F 3 "" H 6675 625 50  0001 C CNN
+	1    6575 875
+	1    0    0    -1
+$EndComp
+Wire Wire Line
+	6575 1300 6575 1225
+Wire Wire Line
+	6875 875  6975 875
+Wire Wire Line
+	3075 850  3075 575
+Wire Wire Line
+	3075 575  5850 575
+Wire Wire Line
+	5850 575  5850 875
+Wire Wire Line
+	5850 875  5975 875
+Connection ~ 3075 850
+Wire Wire Line
+	3075 850  3375 850
+$Comp
+L power:+3V3 #PWR0123
+U 1 1 6375A2DF
+P 7700 750
+F 0 "#PWR0123" H 7700 600 50  0001 C CNN
+F 1 "+3V3" H 7715 923 50  0000 C CNN
+F 2 "" H 7700 750 50  0001 C CNN
+F 3 "" H 7700 750 50  0001 C CNN
+	1    7700 750
+	1    0    0    -1
+$EndComp
+Wire Wire Line
+	7250 875  7700 875
+Wire Wire Line
+	7700 875  7700 750
+$Comp
+L Device:C_Small C1
+U 1 1 63762D32
+P 5975 1075
+F 0 "C1" H 6067 1121 50  0000 L CNN
+F 1 "100nF" H 6067 1030 50  0000 L CNN
+F 2 "Capacitor_SMD:C_0805_2012Metric" H 5975 1075 50  0001 C CNN
+F 3 "~" H 5975 1075 50  0001 C CNN
+	1    5975 1075
+	1    0    0    -1
+$EndComp
+$Comp
+L Device:C_Small C2
+U 1 1 6376314C
+P 6975 1075
+F 0 "C2" H 7067 1121 50  0000 L CNN
+F 1 "100nF" H 7067 1030 50  0000 L CNN
+F 2 "Capacitor_SMD:C_0805_2012Metric" H 6975 1075 50  0001 C CNN
+F 3 "~" H 6975 1075 50  0001 C CNN
+	1    6975 1075
+	1    0    0    -1
+$EndComp
+Wire Wire Line
+	6975 975  6975 875
+Connection ~ 6975 875
+Wire Wire Line
+	6975 875  7050 875
+Wire Wire Line
+	5975 875  5975 975
+Connection ~ 5975 875
+Wire Wire Line
+	5975 875  6275 875
+Wire Wire Line
+	5975 1175 5975 1225
+Wire Wire Line
+	5975 1225 6575 1225
+Connection ~ 6575 1225
+Wire Wire Line
+	6575 1225 6575 1175
+Wire Wire Line
+	6575 1225 6975 1225
+Wire Wire Line
+	6975 1225 6975 1175
+$Comp
+L power:GND #PWR0124
+U 1 1 637823D8
+P 4850 3250
+F 0 "#PWR0124" H 4850 3000 50  0001 C CNN
+F 1 "GND" H 4855 3077 50  0000 C CNN
+F 2 "" H 4850 3250 50  0001 C CNN
+F 3 "" H 4850 3250 50  0001 C CNN
+	1    4850 3250
+	1    0    0    -1
+$EndComp
 $EndSCHEMATC

Commit message: Updates
Connections:
- net VPP_IN is gone; now on net VCC_SLOT: C1.1, U1.40 (VBUS), U4.3 (VI)
Other:
- note added: "+5V for datapack and DC-DC converter"
Changed lines of the file:
@@
 	1    0    0    -1
 $EndComp
+Text GLabel 3375 975  2    50   Input ~ 0
+VCC_SLOT
+Wire Wire Line
+	3375 975  3075 975
+Wire Wire Line
+	3075 975  3075 850
+Text Notes 2775 550  0    50   ~ 0
++5V for datapack and DC-DC converter
 $EndSCHEMATC
