File: pcb/datapack-tool1/datapack-tool1.sch (KiCad schematic (older format))
At the start: 29 parts, among them J1 Conn_01x04_Female, J2 Conn_02x08_Odd_Even, J3 Conn_01x03_Female, M1 P-CHANNEL-MOSFET, SW1 sw, SW2 sw, SW3 sw, U1 Pico, U2 74LS245, U3 74LS245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

Commit message: Updates
Parts:
- R3, R4, R5: value R_Small -> 10k
- R8: value R_Small -> 47k
Changed lines of the file:
@@
 P 9175 4775
 F 0 "R8" H 9234 4821 50  0000 L CNN
-F 1 "R_Small" H 9234 4730 50  0000 L CNN
+F 1 "47k" H 9234 4730 50  0000 L CNN
 F 2 "Resistor_SMD:R_0805_2012Metric" H 9175 4775 50  0001 C CNN
 F 3 "~" H 9175 4775 50  0001 C CNN
@@
 P 3925 6375
 F 0 "R3" H 3984 6421 50  0000 L CNN
-F 1 "R_Small" H 3984 6330 50  0000 L CNN
+F 1 "10k" H 3984 6330 50  0000 L CNN
 F 2 "Resistor_SMD:R_0805_2012Metric" H 3925 6375 50  0001 C CNN
 F 3 "~" H 3925 6375 50  0001 C CNN
@@
 P 4600 6375
 F 0 "R4" H 4659 6421 50  0000 L CNN
-F 1 "R_Small" H 4659 6330 50  0000 L CNN
+F 1 "10k" H 4659 6330 50  0000 L CNN
 F 2 "Resistor_SMD:R_0805_2012Metric" H 4600 6375 50  0001 C CNN
 F 3 "~" H 4600 6375 50  0001 C CNN
@@
 P 5275 6375
 F 0 "R5" H 5334 6421 50  0000 L CNN
-F 1 "R_Small" H 5334 6330 50  0000 L CNN
+F 1 "10k" H 5334 6330 50  0000 L CNN
 F 2 "Resistor_SMD:R_0805_2012Metric" H 5275 6375 50  0001 C CNN
 F 3 "~" H 5275 6375 50  0001 C CNN
