File: pcb/datapack-tool1/datapack-tool1.kicad_pcb (KiCad board)
At the start: 2 copper layers, 139.1 x 63.5 mm, 38 parts, among them J1 Conn_01x04_Female, J2 Conn_02x08_Odd_Even, J3 Conn_01x03_Female, M1 P-CHANNEL-MOSFET, SW1 sw, SW2 sw, SW3 sw, U1 Pico, U2 74LS245, U3 74LS245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

Commit message: Updates
Routing:
- added copper zone on F.Cu, net GND
Changed lines of the file:
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@@
   (segment (start 185.166 130.754) (end 185.12 130.8) (width 0.25) (layer B.Cu) (net 59))
   (segment (start 185.166 122.428) (end 185.166 130.754) (width 0.25) (layer B.Cu) (net 59))
+  (zone (net 1) (net_name GND) (layer F.Cu) (hatch edge 0.508)
+    (connect_pads (clearance 0.508))
+    (min_thickness 0.254)
+    (fill yes (arc_segments 32) (thermal_gap 0.508) (thermal_bridge_width 0.508))
+    (polygon
+      (pts
+        (xy 210.566 167.132) (xy 65.024 166.116) (xy 66.548 99.06) (xy 209.042 98.806)
+      )
+    )
+  )
 )

Commit message: Updates
Parts:
- added C1: 100nF, Capacitor_SMD:C_0805_2012Metric, F.Cu at (174.0, 108.2)
- added C2: 100nF, Capacitor_SMD:C_0805_2012Metric, F.Cu at (181.4, 103.4)
- added JP5: Jumper_NO_Small, Jumper:SolderJumper-2_P1.3mm_Open_TrianglePad1.0x1.5mm, F.Cu at (139.9, 119.6)
- added JP6: Jumper_NO_Small, Jumper:SolderJumper-2_P1.3mm_Open_TrianglePad1.0x1.5mm, F.Cu at (186.7, 113.8)
- added U4: AMS1117-3.3, Package_TO_SOT_SMD:SOT-223-3_TabPin2, F.Cu at (181.4, 108.2)
Connections:
- U1 pad 36: +3V3 -> Net-(JP5-Pad2)
Routing:
- net VPP_IN: track 8.66 -> 49.7 mm, vias 0 -> 2
- net GND: track 438.8 -> 462.9 mm
- net Net-(C2-Pad1): track 0.00 -> 18.7 mm
- net +3V3: track 329.4 -> 336.7 mm
- net Net-(JP5-Pad2): track 0.00 -> 5.25 mm
- removed copper zone on F.Cu, net GND

Commit message: Updates
Parts:
- moved R2 7.74 mm to (192.8, 121.7), turned to 180 degrees
- moved R1 5.01 mm to (192.8, 123.2), turned to 180 degrees
- moved J1 3.04 mm to (190.2, 127.8)
- moved SW1 0.51 mm to (179.8, 157.5)
Connections:
- C1 pad 1: VPP_IN -> VCC_SLOT
- J2 pad 15: (no net) -> VCC_SLOT
- JP11 pad 1: VPP_IN -> VCC_SLOT
- U1 pad 40: VPP_IN -> VCC_SLOT
- U4 pad 3: VPP_IN -> VCC_SLOT
Routing:
- net VCC_SLOT: track 0.00 -> 120.7 mm, vias 0 -> 3
- net VPP_IN: track 49.7 -> 0.00 mm, vias 2 -> 0
- net I2C_SCLK: track 108.8 -> 118.2 mm
- net I2C_SDA: track 119.0 -> 125.3 mm
- net Net-(J1-Pad4): track 12.6 -> 9.52 mm
- net Net-(J1-Pad3): track 13.7 -> 10.7 mm
- net +3V3: track 336.7 -> 334.7 mm
- net GND: track 462.9 -> 463.9 mm

Commit message: Updates
Routing:
- net +3V3: track 334.7 -> 331.9 mm
Other:
- board text added: "3V3"
- board text added: "Datapack reader/Writer Nov 2022 Menadue/Prest V1.0"
- board text added: "GND"
- board text added: "Insert datapack with window upwards or to right."
- board text added: "JP11 DC-DC converter input"
- board text added: "JP12 DC-DC converter output"
- board text added: "JP5: 3V3 from Pico"
- board text added: "JP6:3V3 from regulator"
- board text added: "OLED Power jumpers"
- board text added: "Pin3"
- board text added: "Pin4"
Changed lines of the file:
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@@
   (general
     (thickness 1.6)
-    (drawings 6)
-    (tracks 820)
+    (drawings 24)
+    (tracks 818)
     (zones 0)
     (modules 43)
@@
     (47 F.CrtYd user)
     (48 B.Fab user)
-    (49 F.Fab user)
+    (49 F.Fab user hide)
   )
   (setup
@@
       (outputformat 1)
       (mirror false)
-      (drillshape 1)
+      (drillshape 0)
       (scaleselection 1)
-      (outputdirectory ""))
+      (outputdirectory "fab1/"))
   )
   (net 0 "")
@@
     (tags "CMS SOT")
     (attr smd)
-    (fp_text reference U4 (at 0 -4.5) (layer F.SilkS)
+    (fp_text reference U4 (at -0.254 4.826) (layer F.SilkS)
       (effects (font (size 1 1) (thickness 0.15)))
     )
@@
     (tags "solder jumper open")
     (attr virtual)
-    (fp_text reference JP5 (at 0 -1.8) (layer F.SilkS)
+    (fp_text reference JP5 (at -1.561 2.286) (layer F.SilkS)
       (effects (font (size 1 1) (thickness 0.15)))
     )
@@
     (tags capacitor)
     (attr smd)
-    (fp_text reference C2 (at 0 -1.68) (layer F.SilkS)
+    (fp_text reference C2 (at -4.064 0.508) (layer F.SilkS)
       (effects (font (size 1 1) (thickness 0.15)))
     )
@@
     (tags capacitor)
     (attr smd)
-    (fp_text reference C1 (at 0 -1.68 90) (layer F.SilkS)
+    (fp_text reference C1 (at 3.302 -0.254 90) (layer F.SilkS)
       (effects (font (size 1 1) (thickness 0.15)))
     )
@@
     (tags "solder jumper open")
     (attr virtual)
-    (fp_text reference JP4 (at 0 -1.8) (layer F.SilkS)
+    (fp_text reference JP4 (at -3.525001 -0.097001) (layer F.SilkS)
       (effects (font (size 1 1) (thickness 0.15)))
     )
@@
     (tags "solder jumper open")
     (attr virtual)
-    (fp_text reference JP3 (at 0 -1.8) (layer F.SilkS)
+    (fp_text reference JP3 (at -3.779001 -0.103001) (layer F.SilkS)
       (effects (font (size 1 1) (thickness 0.15)))
     )
@@
     (tags "solder jumper open")
     (attr virtual)
-    (fp_text reference JP2 (at 0 -1.8) (layer F.SilkS)
+    (fp_text reference JP2 (at 2.924999 -0.097001) (layer F.SilkS)
       (effects (font (size 1 1) (thickness 0.15)))
     )
@@
     (tags "solder jumper open")
     (attr virtual)
-    (fp_text reference JP1 (at 0 -1.8) (layer F.SilkS)
+    (fp_text reference JP1 (at 3.178999 -0.103001) (layer F.SilkS)
       (effects (font (size 1 1) (thickness 0.15)))
     )
@@
     (fp_poly (pts (xy -1.5 -14) (xy -3.5 -14) (xy -3.5 -16) (xy -1.5 -16)) (layer Dwgs.User) (width 0.1))
     (fp_poly (pts (xy -1.5 -16.5) (xy -3.5 -16.5) (xy -3.5 -18.5) (xy -1.5 -18.5)) (layer Dwgs.User) (width 0.1))
-    (fp_text user SWDIO (at 5.6 26.2) (layer F.SilkS)
-      (effects (font (size 0.8 0.8) (thickness 0.15)))
-    )
-    (fp_text user SWCLK (at -5.7 26.2) (layer F.SilkS)
+    (fp_text user SWDIO (at -18.166 23.218 90) (layer F.SilkS)
+      (effects (font (size 0.8 0.8) (thickness 0.15)))
+    )
+    (fp_text user SWCLK (at -23.246 22.964 90) (layer F.SilkS)
       (effects (font (size 0.8 0.8) (thickness 0.15)))
     )
@@
       (effects (font (size 0.8 0.8) (thickness 0.15)))
     )
-    (fp_text user 3V3 (at 12.9 -13.9 45) (layer F.SilkS)
-      (effects (font (size 0.8 0.8) (thickness 0.15)))
-    )
-    (fp_text user ADC_VREF (at 14 -12.5 45) (layer F.SilkS)
+    (fp_text user 3V3 (at 4.694 -13.866 45) (layer F.SilkS)
+      (effects (font (size 0.8 0.8) (thickness 0.15)))
+    )
+    (fp_text user ADC_VREF (at 5.202 -11.58 45) (layer F.SilkS)
       (effects (font (size 0.8 0.8) (thickness 0.15)))
     )
@@
     (descr "Through hole angled pin header, 2x08, 2.54mm pitch, 6mm pin length, double rows")
     (tags "Through hole angled pin header THT 2x08 2.54mm double row")
-    (fp_text reference J2 (at 5.655 -2.27) (layer F.SilkS)
+    (fp_text reference J2 (at 7.79 -5.284) (layer F.SilkS)
       (effects (font (size 1 1) (thickness 0.15)))
     )
@@
     (tags SOT-23-6)
     (attr smd)
-    (fp_text reference U6 (at 0 -2.9) (layer F.SilkS)
+    (fp_text reference U6 (at 3.284 -0.754) (layer F.SilkS)
       (effects (font (size 1 1) (thickness 0.15)))
     )
@@
     (tags "SOP SO")
     (attr smd)
-    (fp_text reference U2 (at 0 -7.35) (layer F.SilkS)
+    (fp_text reference U2 (at 3.864 -7.826) (layer F.SilkS)
       (effects (font (size 1 1) (thickness 0.15)))
     )
@@
     (tags resistor)
     (attr smd)
-    (fp_text reference R28 (at 0 -1.65) (layer F.SilkS)
+    (fp_text reference R28 (at 0.092 -1.874) (layer F.SilkS)
       (effects (font (size 1 1) (thickness 0.15)))
     )
@@
     (tags resistor)
     (attr smd)
-    (fp_text reference R18 (at 0 -1.65) (layer F.SilkS)
+    (fp_text reference R18 (at -3.1325 -1.526) (layer F.SilkS)
       (effects (font (size 1 1) (thickness 0.15)))
     )
@@
     (tags resistor)
     (attr smd)
-    (fp_text reference R17 (at 0 -1.65 90) (layer F.SilkS)
+    (fp_text reference R17 (at 0 1.752 90) (layer F.SilkS)
       (effects (font (size 1 1) (thickness 0.15)))
     )
@@
     (tags resistor)
     (attr smd)
-    (fp_text reference R10 (at 0 -1.65) (layer F.SilkS)
+    (fp_text reference R10 (at 0.754 1.776) (layer F.SilkS)
       (effects (font (size 1 1) (thickness 0.15)))
     )
@@
     (tags resistor)
     (attr smd)
-    (fp_text reference R6 (at 0 -1.65 90) (layer F.SilkS)
+    (fp_text reference R6 (at 3.564 -0.108 90) (layer F.SilkS)
       (effects (font (size 1 1) (thickness 0.15)))
     )
@@
     (tags capacitor)
     (attr smd)
-    (fp_text reference R2 (at 0 -1.16) (layer F.SilkS)
+    (fp_text reference R2 (at -2.286 0.254) (layer F.SilkS)
       (effects (font (size 1 1) (thickness 0.15)))
     )
@@
     (tags capacitor)
     (attr smd)
-    (fp_text reference R1 (at 0 -1.16) (layer F.SilkS)
+    (fp_text reference R1 (at -2.286 0) (layer F.SilkS)
       (effects (font (size 1 1) (thickness 0.15)))
     )
@@
     (tags SOT-23)
     (attr smd)
-    (fp_text reference M1 (at 0 -2.5 90) (layer F.SilkS)
+    (fp_text reference M1 (at -0.2 2.51 90) (layer F.SilkS)
       (effects (font (size 1 1) (thickness 0.15)))
     )
@@
     (tags SOD-123)
     (attr smd)
-    (fp_text reference D4 (at 0 -2) (layer F.SilkS)
+    (fp_text reference D4 (at -0.18 2.358) (layer F.SilkS)
       (effects (font (size 1 1) (thickness 0.15)))
     )
@@
     (tags capacitor)
     (attr smd)
-    (fp_text reference C17 (at 0 -1.68) (layer F.SilkS)
+    (fp_text reference C17 (at 3.058 0.05) (layer F.SilkS)
       (effects (font (size 1 1) (thickness 0.15)))
     )
@@
     (tags "capacitor handsolder")
     (attr smd)
-    (fp_text reference C16 (at 0 -2.3) (layer F.SilkS)
+    (fp_text reference C16 (at 0 -2.832) (layer F.SilkS)
       (effects (font (size 1 1) (thickness 0.15)))
     )
@@
     (tags "capacitor handsolder")
     (attr smd)
-    (fp_text reference C15 (at 0 -2.3 90) (layer F.SilkS)
+    (fp_text reference C15 (at -3.704 0.294 180) (layer F.SilkS)
       (effects (font (size 1 1) (thickness 0.15)))
     )
@@
     (tags "capacitor handsolder")
     (attr smd)
-    (fp_text reference C14 (at 0 -2.3 90) (layer F.SilkS)
+    (fp_text reference C14 (at 0 2.704 90) (layer F.SilkS)
       (effects (font (size 1 1) (thickness 0.15)))
     )
@@
       (rotate (xyz 0 0 0))
     )
+  )
+  (gr_text "JP6:3V3 from regulator" (at 197.104 106.172) (layer F.SilkS)
+    (effects (font (size 1 1) (thickness 0.15)))
+  )
+  (gr_text "JP5: 3V3 from Pico" (at 195.834 104.394) (layer F.SilkS)
+    (effects (font (size 1 1) (thickness 0.15)))
+  )
+  (gr_text "OLED Power \njumpers" (at 195.326 116.078) (layer F.SilkS)
+    (effects (font (size 1 1) (thickness 0.15)))
+  )
+  (gr_text "JP12 DC-DC\nconverter output" (at 165.354 103.886) (layer F.SilkS)
+    (effects (font (size 1 1) (thickness 0.15)))
+  )
+  (gr_text "JP11 DC-DC \nconverter input" (at 134.366 103.632) (layer F.SilkS)
+    (effects (font (size 1 1) (thickness 0.15)))
+  )
+  (gr_line (start 76.962 104.14) (end 76.962 107.696) (layer F.SilkS) (width 0.12))
+  (gr_circle (center 73.66 105.918) (end 73.66 104.902) (layer F.SilkS) (width 0.12))
+  (gr_line (start 71.12 107.696) (end 71.12 104.14) (layer F.SilkS) (width 0.12))
+  (gr_line (start 78.232 107.696) (end 71.12 107.696) (layer F.SilkS) (width 0.12))
+  (gr_line (start 78.232 104.14) (end 78.232 107.696) (layer F.SilkS) (width 0.12))
+  (gr_line (start 71.12 104.14) (end 78.232 104.14) (layer F.SilkS) (width 0.12))
+  (gr_text "Insert datapack with window\nupwards or to right." (at 89.662 104.394) (layer F.SilkS)
+    (effects (font (size 1 1) (thickness 0.15)))
+  )
+  (gr_text GND (at 184.404 122.682) (layer F.SilkS)
+    (effects (font (size 1 1) (thickness 0.15)))
+  )
+  (gr_text Pin3 (at 187.452 116.586) (layer F.SilkS)
+    (effects (font (size 1 1) (thickness 0.15)))
+  )
+  (gr_text 3V3 (at 184.404 118.872) (layer F.SilkS)
+    (effects (font (size 1 1) (thickness 0.15)))
+  )
+  (gr_text Pin4 (at 181.102 116.586) (layer F.SilkS)
+    (effects (font (size 1 1) (thickness 0.15)))
+  )
+  (gr_text "Datapack reader/Writer\nNov 2022\nMenadue/Prest\nV1.0" (at 191.262 140.462) (layer F.SilkS)
+    (effects (font (size 1 1) (thickness 0.15)))
+  )
+  (gr_text GND (at 104.394 156.718 90) (layer F.SilkS)
+    (effects (font (size 1 1) (thickness 0.15)))
   )
   (gr_line (start 67.945 163.195) (end 67.945 100.33) (layer Edge.Cuts) (width 0.05))
@@
   (segment (start 193.266 123.19) (end 193.266 123.67) (width 0.25) (layer F.Cu) (net 11))
   (segment (start 193.266 123.19) (end 193.266 121.666) (width 0.25) (layer F.Cu) (net 11))
-  (segment (start 190.246 120.921) (end 190.246 123.698) (width 0.25) (layer F.Cu) (net 11))
-  (segment (start 190.246 123.698) (end 190.246 123.726) (width 0.25) (layer F.Cu) (net 11))
   (segment (start 192.831 120.921) (end 190.246 120.921) (width 0.25) (layer F.Cu) (net 11))
   (segment (start 193.266 121.356) (end 192.831 120.921) (width 0.25) (layer F.Cu) (net 11))

Commit message: Updates
Routing:
- added copper zone on F.Cu, net GND
Changed lines of the file:
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@@
   (segment (start 134.094 119.634) (end 133.99 119.53) (width 0.5) (layer F.Cu) (net 61))
   (segment (start 139.192 119.634) (end 134.094 119.634) (width 0.5) (layer F.Cu) (net 61))
+  (zone (net 1) (net_name GND) (layer F.Cu) (hatch edge 0.508)
+    (connect_pads (clearance 0.508))
+    (min_thickness 0.254)
+    (fill yes (arc_segments 32) (thermal_gap 0.508) (thermal_bridge_width 0.508))
+    (polygon
+      (pts
+        (xy 208.788 165.862) (xy 66.294 164.592) (xy 67.056 99.568) (xy 208.026 99.568)
+      )
+    )
+  )
 )

Commit message: Updates
Parts:
- R3, R4, R5: value R_Small -> 10k
Changed lines of the file:
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@@
     (add_net "Net-(U1-Pad37)")
     (add_net "Net-(U1-Pad39)")
+    (add_net "Net-(U2-Pad19)")
+    (add_net "Net-(U3-Pad11)")
+    (add_net "Net-(U3-Pad12)")
+    (add_net "Net-(U3-Pad13)")
+    (add_net "Net-(U3-Pad7)")
+    (add_net "Net-(U3-Pad8)")
+    (add_net "Net-(U3-Pad9)")
+    (add_net "Net-(U6-Pad6)")
+    (add_net "Net-(XS1-Pad9)")
     (add_net P_SCLK)
     (add_net P_SD0)
@@
       (effects (font (size 1 1) (thickness 0.15)))
     )
-    (fp_text value R_Small (at 0 1.65 90) (layer F.Fab)
+    (fp_text value 10k (at 0 1.65 90) (layer F.Fab)
       (effects (font (size 1 1) (thickness 0.15)))
     )
@@
       (effects (font (size 1 1) (thickness 0.15)))
     )
-    (fp_text value R_Small (at 0 1.65 90) (layer F.Fab)
+    (fp_text value 10k (at 0 1.65 90) (layer F.Fab)
       (effects (font (size 1 1) (thickness 0.15)))
     )
@@
       (effects (font (size 1 1) (thickness 0.15)))
     )
-    (fp_text value R_Small (at 0 1.65 90) (layer F.Fab)
+    (fp_text value 10k (at 0 1.65 90) (layer F.Fab)
       (effects (font (size 1 1) (thickness 0.15)))
     )
@@
   (segment (start 120.535001 159.424999) (end 121.710001 158.249999) (width 0.25) (layer F.Cu) (net 7))
   (segment (start 101.8 160.6) (end 101.8 159.5) (width 0.25) (layer F.Cu) (net 7))
-  (segment (start 134.96 108.4) (end 142.25 108.4) (width 0.5) (layer F.Cu) (net 53))
-  (segment (start 133.99 109.37) (end 134.96 108.4) (width 0.5) (layer F.Cu) (net 53))
-  (segment (start 176.706 110.504) (end 176.466 110.744) (width 0.5) (layer F.Cu) (net 53))
-  (segment (start 178.206 110.504) (end 176.706 110.504) (width 0.5) (layer F.Cu) (net 53))
-  (segment (start 174.876 109.154) (end 173.99 109.154) (width 0.5) (layer F.Cu) (net 53))
-  (segment (start 176.466 110.744) (end 174.876 109.154) (width 0.5) (layer F.Cu) (net 53))
-  (segment (start 142.25 107.5) (end 143.002 106.748) (width 0.5) (layer F.Cu) (net 53))
-  (segment (start 142.25 108.4) (end 142.25 107.5) (width 0.5) (layer F.Cu) (net 53))
-  (via (at 170.18 107.188) (size 0.8) (drill 0.4) (layers F.Cu B.Cu) (net 53))
-  (segment (start 169.68699 106.69499) (end 170.18 107.188) (width 0.5) (layer F.Cu) (net 53))
-  (segment (start 143.05501 106.69499) (end 169.68699 106.69499) (width 0.5) (layer F.Cu) (net 53))
-  (segment (start 143.002 106.748) (end 143.05501 106.69499) (width 0.5) (layer F.Cu) (net 53))
-  (via (at 173.736 110.744) (size 0.8) (drill 0.4) (layers F.Cu B.Cu) (net 53))
-  (segment (start 170.18 107.188) (end 173.736 110.744) (width 0.5) (layer B.Cu) (net 53))
-  (segment (start 173.736 109.408) (end 173.99 109.154) (width 0.5) (layer F.Cu) (net 53))
-  (segment (start 173.736 110.744) (end 173.736 109.408) (width 0.5) (layer F.Cu) (net 53))
   (via (at 80.01 134.112) (size 0.8) (drill 0.4) (layers F.Cu B.Cu) (net 8))
   (segment (start 80.742 133.38) (end 80.01 134.112) (width 0.25) (layer F.Cu) (net 8))
@@
   (segment (start 133.886 157.734) (end 133.99 157.63) (width 0.25) (layer F.Cu) (net 52))
   (segment (start 130.048 157.734) (end 133.886 157.734) (width 0.25) (layer F.Cu) (net 52))
+  (segment (start 134.96 108.4) (end 142.25 108.4) (width 0.5) (layer F.Cu) (net 53))
+  (segment (start 133.99 109.37) (end 134.96 108.4) (width 0.5) (layer F.Cu) (net 53))
+  (segment (start 176.706 110.504) (end 176.466 110.744) (width 0.5) (layer F.Cu) (net 53))
+  (segment (start 178.206 110.504) (end 176.706 110.504) (width 0.5) (layer F.Cu) (net 53))
+  (segment (start 174.876 109.154) (end 173.99 109.154) (width 0.5) (layer F.Cu) (net 53))
+  (segment (start 176.466 110.744) (end 174.876 109.154) (width 0.5) (layer F.Cu) (net 53))
+  (segment (start 142.25 107.5) (end 143.002 106.748) (width 0.5) (layer F.Cu) (net 53))
+  (segment (start 142.25 108.4) (end 142.25 107.5) (width 0.5) (layer F.Cu) (net 53))
+  (via (at 170.18 107.188) (size 0.8) (drill 0.4) (layers F.Cu B.Cu) (net 53))
+  (segment (start 169.68699 106.69499) (end 170.18 107.188) (width 0.5) (layer F.Cu) (net 53))
+  (segment (start 143.05501 106.69499) (end 169.68699 106.69499) (width 0.5) (layer F.Cu) (net 53))
+  (segment (start 143.002 106.748) (end 143.05501 106.69499) (width 0.5) (layer F.Cu) (net 53))
+  (via (at 173.736 110.744) (size 0.8) (drill 0.4) (layers F.Cu B.Cu) (net 53))
+  (segment (start 170.18 107.188) (end 173.736 110.744) (width 0.5) (layer B.Cu) (net 53))
+  (segment (start 173.736 109.408) (end 173.99 109.154) (width 0.5) (layer F.Cu) (net 53))
+  (segment (start 173.736 110.744) (end 173.736 109.408) (width 0.5) (layer F.Cu) (net 53))
   (via (at 129.54 132.842) (size 0.8) (drill 0.4) (layers F.Cu B.Cu) (net 53))
   (segment (start 128.976999 133.405001) (end 129.54 132.842) (width 0.25) (layer F.Cu) (net 53))
