File: pcb/datapack-tool1/usb.sch (KiCad schematic (older format))
At the start: 12 parts, among them U6 Regulator_Switching_MT3608

Commit message: Updates
Parts:
- added R10, R9: R_Small, Resistor_SMD:R_0805_2012Metric, symbol Device:R_Small
Connections:
- net GND: now also R10.2
- net at R17.2, R18.1, U6.3 (FB): now also R9.1
- net at R18.2, R28.1: now also R10.1, R9.2
Changed lines of the file:
@@
 $Descr A4 11693 8268
 encoding utf-8
-Sheet 5 2
+Sheet 2 2
 Title "Psion Organiser 2 USB Adapter"
 Date ""
@@
 $EndComp
 Wire Wire Line
-	3500 3550 4500 3550
+	3500 3550 4225 3550
 Wire Wire Line
 	4500 3350 4500 3550
@@
 Connection ~ 4500 3550
 Wire Wire Line
-	4500 3800 4500 3875
+	4500 3800 4500 3825
 Wire Wire Line
 	2500 4150 3200 4150
@@
 Connection ~ 3200 4150
 Wire Wire Line
-	3200 4150 4500 4150
+	3200 4150 4225 4150
 Wire Wire Line
 	3200 3750 3200 4150
@@
 	6300 3550 6300 4150
 Connection ~ 5875 4150
+$Comp
+L Device:R_Small R9
+U 1 1 636AA642
+P 4225 3675
+F 0 "R9" H 4284 3721 50  0000 L CNN
+F 1 "R_Small" H 4284 3630 50  0000 L CNN
+F 2 "Resistor_SMD:R_0805_2012Metric" H 4225 3675 50  0001 C CNN
+F 3 "~" H 4225 3675 50  0001 C CNN
+	1    4225 3675
+	1    0    0    -1
+$EndComp
+$Comp
+L Device:R_Small R10
+U 1 1 636AB08C
+P 4225 3975
+F 0 "R10" H 4284 4021 50  0000 L CNN
+F 1 "R_Small" H 4284 3930 50  0000 L CNN
+F 2 "Resistor_SMD:R_0805_2012Metric" H 4225 3975 50  0001 C CNN
+F 3 "~" H 4225 3975 50  0001 C CNN
+	1    4225 3975
+	1    0    0    -1
+$EndComp
+Wire Wire Line
+	4225 3575 4225 3550
+Connection ~ 4225 3550
+Wire Wire Line
+	4225 3550 4500 3550
+Wire Wire Line
+	4225 3775 4225 3825
+Wire Wire Line
+	4225 4075 4225 4150
+Connection ~ 4225 4150
+Wire Wire Line
+	4225 4150 4500 4150
+Wire Wire Line
+	4225 3825 4500 3825
+Connection ~ 4225 3825
+Wire Wire Line
+	4225 3825 4225 3875
+Connection ~ 4500 3825
+Wire Wire Line
+	4500 3825 4500 3875
 $EndSCHEMATC

Commit message: Updates
Parts:
- renumbered C14 to C15, C15 to C16, C16 to C17, C17 to C18, D4 to D6, JP11 to JP12, JP12 to JP13, R9 to R23, R10 to R24, R17 to R25, R18 to R26, R28 to R27, U6 to U11
Changed lines of the file:
@@
 $Descr A4 11693 8268
 encoding utf-8
-Sheet 2 2
+Sheet 2 4
 Title "Psion Organiser 2 USB Adapter"
 Date ""
@@
 AR Path="/630E8640" Ref="R?"  Part="1"
 AR Path="/630BAFD1/630E8640" Ref="R?"  Part="1"
-AR Path="/630E4C46/630E8640" Ref="R18"  Part="1"
-AR Path="/63706713/630E8640" Ref="R18"  Part="1"
-F 0 "R18" H 4559 3746 50  0000 L CNN
+AR Path="/630E4C46/630E8640" Ref="R?"  Part="1"
+AR Path="/63706713/630E8640" Ref="R?"  Part="1"
+AR Path="/6593F8B7/63706713/630E8640" Ref="R26"  Part="1"
+F 0 "R26" H 4559 3746 50  0000 L CNN
 F 1 "????" H 4559 3655 50  0000 L CNN
 F 2 "Resistor_SMD:R_0805_2012Metric" H 4500 3700 50  0001 C CNN
@@
 AR Path="/630E8646" Ref="C?"  Part="1"
 AR Path="/630BAFD1/630E8646" Ref="C?"  Part="1"
-AR Path="/630E4C46/630E8646" Ref="C14"  Part="1"
-AR Path="/63706713/630E8646" Ref="C14"  Part="1"
-F 0 "C14" H 2592 3846 50  0000 L CNN
+AR Path="/630E4C46/630E8646" Ref="C?"  Part="1"
+AR Path="/63706713/630E8646" Ref="C?"  Part="1"
+AR Path="/6593F8B7/63706713/630E8646" Ref="C15"  Part="1"
+F 0 "C15" H 2592 3846 50  0000 L CNN
 F 1 "22uF" H 2592 3755 50  0000 L CNN
 F 2 "Capacitor_SMD:C_1210_3225Metric_Pad1.33x2.70mm_HandSolder" H 2500 3800 50  0001 C CNN
@@
 AR Path="/630E864C" Ref="C?"  Part="1"
 AR Path="/630BAFD1/630E864C" Ref="C?"  Part="1"
-AR Path="/630E4C46/630E864C" Ref="C15"  Part="1"
-AR Path="/63706713/630E864C" Ref="C15"  Part="1"
-F 0 "C15" H 5242 3646 50  0000 L CNN
+AR Path="/630E4C46/630E864C" Ref="C?"  Part="1"
+AR Path="/63706713/630E864C" Ref="C?"  Part="1"
+AR Path="/6593F8B7/63706713/630E864C" Ref="C16"  Part="1"
+F 0 "C16" H 5242 3646 50  0000 L CNN
 F 1 "22uF" H 5242 3555 50  0000 L CNN
 F 2 "Capacitor_SMD:C_1210_3225Metric_Pad1.33x2.70mm_HandSolder" H 5150 3600 50  0001 C CNN
@@
 AR Path="/630E8652" Ref="L?"  Part="1"
 AR Path="/630BAFD1/630E8652" Ref="L?"  Part="1"
-AR Path="/630E4C46/630E8652" Ref="L1"  Part="1"
-AR Path="/63706713/630E8652" Ref="L1"  Part="1"
+AR Path="/630E4C46/630E8652" Ref="L?"  Part="1"
+AR Path="/63706713/630E8652" Ref="L?"  Part="1"
+AR Path="/6593F8B7/63706713/630E8652" Ref="L1"  Part="1"
 F 0 "L1" H 3200 3165 50  0000 C CNN
 F 1 "22uH" H 3200 3074 50  0000 C CNN
@@
 AR Path="/630E8673" Ref="R?"  Part="1"
 AR Path="/630BAFD1/630E8673" Ref="R?"  Part="1"
-AR Path="/630E4C46/630E8673" Ref="R17"  Part="1"
-AR Path="/63706713/630E8673" Ref="R17"  Part="1"
-F 0 "R17" H 4559 3296 50  0000 L CNN
+AR Path="/630E4C46/630E8673" Ref="R?"  Part="1"
+AR Path="/63706713/630E8673" Ref="R?"  Part="1"
+AR Path="/6593F8B7/63706713/630E8673" Ref="R25"  Part="1"
+F 0 "R25" H 4559 3296 50  0000 L CNN
 F 1 "100k" H 4559 3205 50  0000 L CNN
 F 2 "Resistor_SMD:R_0805_2012Metric" H 4500 3250 50  0001 C CNN
@@
 AR Path="/630E867A" Ref="JP?"  Part="1"
 AR Path="/630BAFD1/630E867A" Ref="JP?"  Part="1"
-AR Path="/630E4C46/630E867A" Ref="JP12"  Part="1"
-AR Path="/63706713/630E867A" Ref="JP12"  Part="1"
-F 0 "JP12" H 5500 3155 50  0000 C CNN
+AR Path="/630E4C46/630E867A" Ref="JP?"  Part="1"
+AR Path="/63706713/630E867A" Ref="JP?"  Part="1"
+AR Path="/6593F8B7/63706713/630E867A" Ref="JP13"  Part="1"
+F 0 "JP13" H 5500 3155 50  0000 C CNN
 F 1 "SolderJumper_2_Open" H 5500 3064 50  0000 C CNN
 F 2 "psion_org_2:SolderJumper-2_P1.3mm_Open_Pad0.8x0.8mm" H 5500 2950 50  0001 C CNN
@@
 AR Path="/630E8684" Ref="U?"  Part="1"
 AR Path="/630BAFD1/630E8684" Ref="U?"  Part="1"
-AR Path="/630E4C46/630E8684" Ref="U6"  Part="1"
-AR Path="/63706713/630E8684" Ref="U6"  Part="1"
-F 0 "U6" H 3200 3817 50  0000 C CNN
+AR Path="/630E4C46/630E8684" Ref="U?"  Part="1"
+AR Path="/63706713/630E8684" Ref="U?"  Part="1"
+AR Path="/6593F8B7/63706713/630E8684" Ref="U11"  Part="1"
+F 0 "U11" H 3200 3817 50  0000 C CNN
 F 1 "Regulator_Switching_MT3608" H 3200 3726 50  0000 C CNN
 F 2 "Package_TO_SOT_SMD:SOT-23-6" H 3250 3200 50  0001 L CIN
@@
 P 3750 2950
 AR Path="/630BAFD1/630E868A" Ref="D?"  Part="1"
-AR Path="/630E4C46/630E868A" Ref="D4"  Part="1"
-AR Path="/63706713/630E868A" Ref="D4"  Part="1"
-F 0 "D4" H 3750 2734 50  0000 C CNN
+AR Path="/630E4C46/630E868A" Ref="D?"  Part="1"
+AR Path="/63706713/630E868A" Ref="D?"  Part="1"
+AR Path="/6593F8B7/63706713/630E868A" Ref="D6"  Part="1"
+F 0 "D6" H 3750 2734 50  0000 C CNN
 F 1 "SS36" H 3750 2825 50  0000 C CNN
 F 2 "Diode_SMD:D_SOD-123" H 3750 2950 50  0001 C CNN
@@
 AR Path="/630E8691" Ref="C?"  Part="1"
 AR Path="/630BAFD1/630E8691" Ref="C?"  Part="1"
-AR Path="/630E4C46/630E8691" Ref="C16"  Part="1"
-AR Path="/63706713/630E8691" Ref="C16"  Part="1"
-F 0 "C16" H 5967 3496 50  0000 L CNN
+AR Path="/630E4C46/630E8691" Ref="C?"  Part="1"
+AR Path="/63706713/630E8691" Ref="C?"  Part="1"
+AR Path="/6593F8B7/63706713/630E8691" Ref="C17"  Part="1"
+F 0 "C17" H 5967 3496 50  0000 L CNN
 F 1 "10uF" H 5967 3405 50  0000 L CNN
 F 2 "Capacitor_SMD:C_1210_3225Metric_Pad1.33x2.70mm_HandSolder" H 5875 3450 50  0001 C CNN
@@
 AR Path="/630E8697" Ref="C?"  Part="1"
 AR Path="/630BAFD1/630E8697" Ref="C?"  Part="1"
-AR Path="/630E4C46/630E8697" Ref="C17"  Part="1"
-AR Path="/63706713/630E8697" Ref="C17"  Part="1"
-F 0 "C17" H 6392 3496 50  0000 L CNN
+AR Path="/630E4C46/630E8697" Ref="C?"  Part="1"
+AR Path="/63706713/630E8697" Ref="C?"  Part="1"
+AR Path="/6593F8B7/63706713/630E8697" Ref="C18"  Part="1"
+F 0 "C18" H 6392 3496 50  0000 L CNN
 F 1 "100nF" H 6392 3405 50  0000 L CNN
 F 2 "Capacitor_SMD:C_0805_2012Metric" H 6300 3450 50  0001 C CNN
@@
 P 2075 2375
 AR Path="/630BAFD1/630E86AA" Ref="JP?"  Part="1"
-AR Path="/630E4C46/630E86AA" Ref="JP11"  Part="1"
-AR Path="/63706713/630E86AA" Ref="JP11"  Part="1"
-F 0 "JP11" H 2075 2560 50  0000 C CNN
+AR Path="/630E4C46/630E86AA" Ref="JP?"  Part="1"
+AR Path="/63706713/630E86AA" Ref="JP?"  Part="1"
+AR Path="/6593F8B7/63706713/630E86AA" Ref="JP12"  Part="1"
+F 0 "JP12" H 2075 2560 50  0000 C CNN
 F 1 "Jumper_NO_Small" H 2075 2469 50  0000 C CNN
 F 2 "psion_org_2:SolderJumper-2_P1.3mm_Open_Pad0.8x0.8mm" H 2075 2375 50  0001 C CNN
@@
 P 3200 4225
 AR Path="/630BAFD1/630E86BF" Ref="#PWR?"  Part="1"
-AR Path="/630E4C46/630E86BF" Ref="#PWR022"  Part="1"
-AR Path="/63706713/630E86BF" Ref="#PWR022"  Part="1"
-F 0 "#PWR022" H 3200 3975 50  0001 C CNN
+AR Path="/630E4C46/630E86BF" Ref="#PWR?"  Part="1"
+AR Path="/63706713/630E86BF" Ref="#PWR?"  Part="1"
+AR Path="/6593F8B7/63706713/630E86BF" Ref="#PWR066"  Part="1"
+F 0 "#PWR066" H 3200 3975 50  0001 C CNN
 F 1 "GND" H 3205 4052 50  0000 C CNN
 F 2 "" H 3200 4225 50  0001 C CNN
@@
 AR Path="/6320ACB0" Ref="R?"  Part="1"
 AR Path="/630BAFD1/6320ACB0" Ref="R?"  Part="1"
-AR Path="/630E4C46/6320ACB0" Ref="R28"  Part="1"
-AR Path="/63706713/6320ACB0" Ref="R28"  Part="1"
-F 0 "R28" H 4559 4021 50  0000 L CNN
+AR Path="/630E4C46/6320ACB0" Ref="R?"  Part="1"
+AR Path="/63706713/6320ACB0" Ref="R?"  Part="1"
+AR Path="/6593F8B7/63706713/6320ACB0" Ref="R27"  Part="1"
+F 0 "R27" H 4559 4021 50  0000 L CNN
 F 1 "???????????" H 4559 3930 50  0000 L CNN
 F 2 "Resistor_SMD:R_0805_2012Metric" H 4500 3975 50  0001 C CNN
@@
 Connection ~ 5875 4150
 $Comp
-L Device:R_Small R9
+L Device:R_Small R23
 U 1 1 636AA642
 P 4225 3675
-F 0 "R9" H 4284 3721 50  0000 L CNN
+F 0 "R23" H 4284 3721 50  0000 L CNN
 F 1 "R_Small" H 4284 3630 50  0000 L CNN
 F 2 "Resistor_SMD:R_0805_2012Metric" H 4225 3675 50  0001 C CNN
@@
 $EndComp
 $Comp
-L Device:R_Small R10
+L Device:R_Small R24
 U 1 1 636AB08C
 P 4225 3975
-F 0 "R10" H 4284 4021 50  0000 L CNN
+F 0 "R24" H 4284 4021 50  0000 L CNN
 F 1 "R_Small" H 4284 3930 50  0000 L CNN
 F 2 "Resistor_SMD:R_0805_2012Metric" H 4225 3975 50  0001 C CNN
